File: DemoPCB.kicad_pcb (KiCad board)
At the start: 2 copper layers, 36.8 x 16.5 mm, 7 parts, among them J1 Conn_01x02, J2 Conn_01x02, U1 L7805

Commit message: second fix
fixed a few things
Parts:
- J1, J2: footprint Connector_PinHeader_2.54mm:PinHeader_1x02_P2.54mm_Horizontal -> Connector_PinHeader_2.54mm:PinHeader_1x02_P2.54mm_Vertical
- U1: footprint Package_TO_SOT_THT:TO-92 -> Package_TO_SOT_THT:TO-220-3_Horizontal_TabDown
Routing:
- net V_OUT: track 26.6 -> 24.7 mm

Commit message: first final release
Parts:
- K1: renamed from J1; moved to F.Cu
- K2: renamed from J2; moved to F.Cu
- moved IC1 1.05 mm to (41.9, 18.3)
- turned K1 to 270 degrees
- turned K2 to 90 degrees
- renumbered U1 to IC1
Routing:
- net V_IN: track 22.8 -> 21.2 mm
